File: design_files/ASD2302.brd (EAGLE design)
At the start: 22.5 x 21.3 mm, 24 parts, among them J1 DF12-32-DP, J2 DF12-32-DS, J3 SM02B-SRSS, J4 SM02B-SRSS, J5 SM02B-SRSS, J6 961102, J7 961102, J8 961102, U3 DRV8837, U4 DRV8837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

Commit message: Update format
Other:
- board text added: "TinyCircuits.com"
- board text removed: "Tiny-Circuits.com"
